Commit message: fix: changed mass to be small and added small inertia values for fingertips to fix bug in simulator

File: assets/p50/p50.urdf (robot description, URDF)
Before this commit: robot p50_autoconverted, 27 links, 26 joints
Links:
- link index_fingertip: mass 6.165375582669709e-09 -> 1e-4
- link middle_fingertip: mass 6.165375582669709e-09 -> 1e-4
- link pinky_fingertip: mass 6.165375582669709e-09 -> 1e-4
- link ring_fingertip: mass 6.165375582669709e-09 -> 1e-4
- link thumb_fingertip: mass 6.165375582669709e-09 -> 1e-4

Commit message: fix: commented out <collision> tags to prevent segfault errors

File: assets/p50/p50.urdf (robot description, URDF)
Before this commit: robot p50_autoconverted, 27 links, 26 joints
Links:
- link base_link: geometry visual mesh filename=meshes/visual/base_link.stl scale=0.001 0.001 0.001
- link index_dp: geometry visual mesh filename=meshes/visual/index_dp.stl scale=0.001 0.001 0.001
- link index_fingertip: geometry visual mesh filename=meshes/visual/index_fingertip.stl scale=0.001 0.001 0.001
- link index_mcp: geometry visual mesh filename=meshes/visual/index_mcp.stl scale=0.001 0.001 0.001
- link index_mp: geometry visual mesh filename=meshes/visual/index_mp.stl scale=0.001 0.001 0.001
- link index_pp: geometry visual mesh filename=meshes/visual/index_pp.stl scale=0.001 0.001 0.001
- link middle_dp: geometry visual mesh filename=meshes/visual/middle_dp.stl scale=0.001 0.001 0.001
- link middle_fingertip: geometry visual mesh filename=meshes/visual/middle_fingertip.stl scale=0.001 0.001 0.001
- link middle_mcp: geometry visual mesh filename=meshes/visual/middle_mcp.stl scale=0.001 0.001 0.001
- link middle_mp: geometry visual mesh filename=meshes/visual/middle_mp.stl scale=0.001 0.001 0.001
- link middle_pp: geometry visual mesh filename=meshes/visual/middle_pp.stl scale=0.001 0.001 0.001
- link pinky_dp: geometry visual mesh filename=meshes/visual/pinky_dp.stl scale=0.001 0.001 0.001
- link pinky_fingertip: geometry visual mesh filename=meshes/visual/pinky_fingertip.stl scale=0.001 0.001 0.001
- link pinky_mcp: geometry visual mesh filename=meshes/visual/pinky_mcp.stl scale=0.001 0.001 0.001
- link pinky_mp: geometry visual mesh filename=meshes/visual/pinky_mp.stl scale=0.001 0.001 0.001
- link pinky_pp: geometry visual mesh filename=meshes/visual/pinky_pp.stl scale=0.001 0.001 0.001
- link ring_dp: geometry visual mesh filename=meshes/visual/ring_dp.stl scale=0.001 0.001 0.001
- link ring_fingertip: geometry visual mesh filename=meshes/visual/ring_fingertip.stl scale=0.001 0.001 0.001
- link ring_mcp: geometry visual mesh filename=meshes/visual/ring_mcp.stl scale=0.001 0.001 0.001
- link ring_mp: geometry visual mesh filename=meshes/visual/ring_mp.stl scale=0.001 0.001 0.001
- link ring_pp: geometry visual mesh filename=meshes/visual/ring_pp.stl scale=0.001 0.001 0.001
- link thumb_cmc: geometry visual mesh filename=meshes/visual/thumb_cmc.stl scale=0.001 0.001 0.001
- link thumb_dp: geometry visual mesh filename=meshes/visual/thumb_dp.stl scale=0.001 0.001 0.001
- link thumb_fingertip: geometry visual mesh filename=meshes/visual/thumb_fingertip.stl scale=0.001 0.001 0.001
- link thumb_mp: geometry visual mesh filename=meshes/visual/thumb_mp.stl scale=0.001 0.001 0.001
- link thumb_pp: geometry visual mesh filename=meshes/visual/thumb_pp.stl scale=0.001 0.001 0.001
